File: CAN_Transceiver.kicad_sch (KiCad schematic)
At the start: 3 parts, among them IC1 TJA1441AT

Commit message: ver1.00
Parts:
- C3: renamed from C1; footprint (none) -> Capacitor_SMD:C_0603_1608Metric
- C4: renamed from C2; footprint (none) -> Capacitor_SMD:C_0603_1608Metric
- IC1: footprint SOIC127P600X175-8N -> TJA1441AT:SOIC127P600X175-8N
Changed lines of the file:
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@@
 		(on_board yes)
 		(dnp no)
-		(property "Reference" "C1"
+		(property "Reference" "C3"
 			(at 107.696 71.628 0)
 			(effects
@@
 			)
 		)
-		(property "Footprint" ""
+		(property "Footprint" "Capacitor_SMD:C_0603_1608Metric"
 			(at 112.7252 77.47 0)
 			(effects
@@
 			(project "rm_controller_hardware"
 				(path "/35e8a876-55b4-4d5a-8094-d621f011ebeb/46bc1938-3108-4b90-9a29-7d2ec265e9a5"
+					(reference "C5")
+					(unit 1)
+				)
+				(path "/35e8a876-55b4-4d5a-8094-d621f011ebeb/98a37396-8194-437e-9c8d-2eac45dd7a3d"
 					(reference "C3")
-					(unit 1)
-				)
-				(path "/35e8a876-55b4-4d5a-8094-d621f011ebeb/98a37396-8194-437e-9c8d-2eac45dd7a3d"
-					(reference "C1")
 					(unit 1)
 				)
@@
 		(dnp no)
 		(fields_autoplaced yes)
-		(property "Reference" "#PWR09"
+		(property "Reference" "#PWR019"
 			(at 165.1 86.36 0)
 			(effects
@@
 			(project "rm_controller_hardware"
 				(path "/35e8a876-55b4-4d5a-8094-d621f011ebeb/46bc1938-3108-4b90-9a29-7d2ec265e9a5"
-					(reference "#PWR014")
-					(unit 1)
-				)
-				(path "/35e8a876-55b4-4d5a-8094-d621f011ebeb/98a37396-8194-437e-9c8d-2eac45dd7a3d"
-					(reference "#PWR09")
+					(reference "#PWR024")
+					(unit 1)
+				)
+				(path "/35e8a876-55b4-4d5a-8094-d621f011ebeb/98a37396-8194-437e-9c8d-2eac45dd7a3d"
+					(reference "#PWR019")
 					(unit 1)
 				)
@@
 		(dnp no)
 		(fields_autoplaced yes)
-		(property "Reference" "#PWR06"
+		(property "Reference" "#PWR016"
 			(at 105.41 66.04 0)
 			(effects
@@
 			(project "rm_controller_hardware"
 				(path "/35e8a876-55b4-4d5a-8094-d621f011ebeb/46bc1938-3108-4b90-9a29-7d2ec265e9a5"
-					(reference "#PWR011")
-					(unit 1)
-				)
-				(path "/35e8a876-55b4-4d5a-8094-d621f011ebeb/98a37396-8194-437e-9c8d-2eac45dd7a3d"
-					(reference "#PWR06")
+					(reference "#PWR021")
+					(unit 1)
+				)
+				(path "/35e8a876-55b4-4d5a-8094-d621f011ebeb/98a37396-8194-437e-9c8d-2eac45dd7a3d"
+					(reference "#PWR016")
 					(unit 1)
 				)
@@
 		(on_board yes)
 		(dnp no)
-		(property "Reference" "C2"
+		(property "Reference" "C4"
 			(at 154.686 74.168 0)
 			(effects
@@
 			)
 		)
-		(property "Footprint" ""
+		(property "Footprint" "Capacitor_SMD:C_0603_1608Metric"
 			(at 159.7152 80.01 0)
 			(effects
@@
 			(project "rm_controller_hardware"
 				(path "/35e8a876-55b4-4d5a-8094-d621f011ebeb/46bc1938-3108-4b90-9a29-7d2ec265e9a5"
+					(reference "C6")
+					(unit 1)
+				)
+				(path "/35e8a876-55b4-4d5a-8094-d621f011ebeb/98a37396-8194-437e-9c8d-2eac45dd7a3d"
 					(reference "C4")
-					(unit 1)
-				)
-				(path "/35e8a876-55b4-4d5a-8094-d621f011ebeb/98a37396-8194-437e-9c8d-2eac45dd7a3d"
-					(reference "C2")
 					(unit 1)
 				)
@@
 		(dnp no)
 		(fields_autoplaced yes)
-		(property "Reference" "#PWR05"
+		(property "Reference" "#PWR015"
 			(at 100.33 86.36 0)
 			(effects
@@
 			(project "rm_controller_hardware"
 				(path "/35e8a876-55b4-4d5a-8094-d621f011ebeb/46bc1938-3108-4b90-9a29-7d2ec265e9a5"
-					(reference "#PWR010")
-					(unit 1)
-				)
-				(path "/35e8a876-55b4-4d5a-8094-d621f011ebeb/98a37396-8194-437e-9c8d-2eac45dd7a3d"
-					(reference "#PWR05")
+					(reference "#PWR020")
+					(unit 1)
+				)
+				(path "/35e8a876-55b4-4d5a-8094-d621f011ebeb/98a37396-8194-437e-9c8d-2eac45dd7a3d"
+					(reference "#PWR015")
 					(unit 1)
 				)
@@
 		(dnp no)
 		(fields_autoplaced yes)
-		(property "Reference" "#PWR08"
+		(property "Reference" "#PWR018"
 			(at 158.75 86.36 0)
 			(effects
@@
 			(project "rm_controller_hardware"
 				(path "/35e8a876-55b4-4d5a-8094-d621f011ebeb/46bc1938-3108-4b90-9a29-7d2ec265e9a5"
-					(reference "#PWR013")
-					(unit 1)
-				)
-				(path "/35e8a876-55b4-4d5a-8094-d621f011ebeb/98a37396-8194-437e-9c8d-2eac45dd7a3d"
-					(reference "#PWR08")
+					(reference "#PWR023")
+					(unit 1)
+				)
+				(path "/35e8a876-55b4-4d5a-8094-d621f011ebeb/98a37396-8194-437e-9c8d-2eac45dd7a3d"
+					(reference "#PWR018")
 					(unit 1)
 				)
@@
 		(dnp no)
 		(fields_autoplaced yes)
-		(property "Reference" "#PWR07"
+		(property "Reference" "#PWR017"
 			(at 152.4 68.58 0)
 			(effects
@@
 			(project "rm_controller_hardware"
 				(path "/35e8a876-55b4-4d5a-8094-d621f011ebeb/46bc1938-3108-4b90-9a29-7d2ec265e9a5"
-					(reference "#PWR012")
-					(unit 1)
-				)
-				(path "/35e8a876-55b4-4d5a-8094-d621f011ebeb/98a37396-8194-437e-9c8d-2eac45dd7a3d"
-					(reference "#PWR07")
+					(reference "#PWR022")
+					(unit 1)
+				)
+				(path "/35e8a876-55b4-4d5a-8094-d621f011ebeb/98a37396-8194-437e-9c8d-2eac45dd7a3d"
+					(reference "#PWR017")
 					(unit 1)
 				)
@@
 			)
 		)
-		(property "Footprint" "SOIC127P600X175-8N"
+		(property "Footprint" "TJA1441AT:SOIC127P600X175-8N"
 			(at 147.32 62.23 0)
 			(effects
