File: CAN_Transceiver.kicad_sch (KiCad schematic)
At the start: 3 parts, among them IC1 TJA1441AT

Commit message: Ver1.1
Parts:
- C3, C4: footprint Capacitor_SMD:C_0603_1608Metric -> Capacitor_SMD:C_0603_1608Metric_Pad1.08x0.95mm_HandSolder
- IC1: footprint TJA1441AT:SOIC127P600X175-8N -> tja1441at:SO8_SOT96-1_NXP
