File: MCU_STM32G473CETx.kicad_sch (KiCad schematic)
At the start: 12 parts, among them J6 STLink/v3, SW1 SW_Push, U1 STM32G473CETx

Commit message: ver1.00
Parts:
- added D1, D2, D3: LED_GREEN, LED_SMD:LED_0603_1608Metric_Pad1.05x0.95mm_HandSolder, symbol Device:LED_Small
- added R1, R2, R3: 330, Resistor_SMD:R_0603_1608Metric_Pad0.98x0.95mm_HandSolder, symbol Device:R_Small
- added R4: 10k, Resistor_SMD:R_0603_1608Metric_Pad0.98x0.95mm_HandSolder, symbol Device:R_Small
- C10: renamed from C8; footprint (none) -> Capacitor_SMD:C_0603_1608Metric
- C11: renamed from C9; footprint (none) -> Capacitor_SMD:C_0603_1608Metric
- C12: renamed from C10; footprint (none) -> Capacitor_SMD:C_0603_1608Metric
- C13: renamed from C11; footprint (none) -> Capacitor_SMD:C_0603_1608Metric
- C14: renamed from C12; footprint (none) -> Capacitor_SMD:C_0603_1608Metric
- C15: renamed from C13; footprint (none) -> Capacitor_SMD:C_0603_1608Metric
- C7: renamed from C5; footprint (none) -> Capacitor_SMD:C_0603_1608Metric
- C8: renamed from C6; footprint (none) -> Capacitor_SMD:C_0603_1608Metric
- C9: renamed from C7; footprint (none) -> Capacitor_SMD:C_0603_1608Metric
- J21: renamed from J6; footprint 3220-14-0100-00:CONN14_3220-14_CNC -> footprints:CONN14_3220-14_CNC
- SW1: footprint (none) -> d_robo_lib:TVAF06-A020B-R
- renumbered U1 to U2
Connections:
- net +3V3 is gone; now on net +3.3V: J21.3 (Pin_3)
- net +3.3V: now also R4.1
- net GND: now also J21.7 (Pin_7), D1.1 (K), D2.1 (K), D3.1 (K)
- net NRST: now also R4.2
- net LED_1: now reaches U2.2 (PC13)
- net LED_1: now also R1.1
- net LED_2: now reaches U2.3 (PC14)
- net LED_2: now also R2.1
- net I2C_SDL: now reaches U2.39 (PA15)
- net LED_3: now reaches U2.4 (PC15)
- net LED_3: now also R3.1
- net I2C_SDA: now reaches U2.44 (PB7)
- new net: D1.2 (A), R1.2
- new net: D3.2 (A), R3.2
- new net: D2.2 (A), R2.2
- no-connect marks 37 -> 31
