File: rm_controller_hardware.kicad_pcb (KiCad board)
At the start: 2 copper layers, 90 x 65 mm, 49 parts, among them IC1 TJA1441AT, IC2 TJA1441AT, J1 XT60PW-M_Horizontal, J10 SM02B-GHS-TB, J11 SM02B-GHS-TB, J12 SM02B-GHS-TB, J13 SM02B-GHS-TB, J14 SM02B-GHS-TB, J15 SM02B-GHS-TB, J16 SM02B-GHS-TB, J17 SM02B-GHS-TB, J18 RJ45, J19 Conn_01x02_Pin, J2 XT30PW-F_Horizontal, J20 RJ45, J21 STLink/v3, J22 Conn_01x04_Pin, J3 XT30PW-F_Horizontal, J4 XT30PW-F_Horizontal, J5 XT30PW-F_Horizontal, J6 XT30PW-F_Horizontal, J7 XT30PW-F_Horizontal, J8 XT30PW-F_Horizontal, J9 XT30PW-F_Horizontal, SW1 SW_Push, U1 BU33SD5WG-TR, U2 STM32G473CETx

Commit message: Ver1.1
Parts:
- added C16: 0.47μ, Capacitor_SMD:C_0603_1608Metric_Pad1.08x0.95mm_HandSolder, F.Cu at (115.0, 89.9)
- added Q3: RD3L07BBGTL1, y-robo_footprint:TO252-3_ROM, F.Cu at (121.2, 89.4)
- added R5: 100k, Resistor_SMD:R_0603_1608Metric_Pad0.98x0.95mm_HandSolder, F.Cu at (115.0, 92.8)
- added R6: 100k, Resistor_SMD:R_0603_1608Metric_Pad0.98x0.95mm_HandSolder, F.Cu at (115.0, 95.7)
- C3, C4, C5, C6: footprint Capacitor_SMD:C_0603_1608Metric -> Capacitor_SMD:C_0603_1608Metric_Pad1.08x0.95mm_HandSolder
- IC1, IC2: footprint TJA1441AT:SOIC127P600X175-8N -> tja1441at:SO8_SOT96-1_NXP
Connections:
- J2 pad 1: GNDPWR -> GND1
- J3 pad 1: GNDPWR -> GND1
- J4 pad 1: GNDPWR -> GND1
- J5 pad 1: GNDPWR -> GND1
- J6 pad 1: GNDPWR -> GND1
- J7 pad 1: GNDPWR -> GND1
- J8 pad 1: GNDPWR -> GND1
- J9 pad 1: GNDPWR -> GND1
Routing:
- net GND1: track 0.00 -> 19.5 mm
- net Net-(Q3-G): track 0.00 -> 11.2 mm
- net VSS: vias 184 -> 178
- added copper zone on B.Cu, net GND1
- added copper zone on F.Cu, net GNDPWR
- removed copper zone on B.Cu, net GNDPWR
Other:
- board text added: "rm_controller_hardware ver 1.10 nityc 2026"
- board text removed: "rm_controller_hardware ver 1.00 nityc 2025"
