File: rm_controller_hardware.kicad_sch (KiCad schematic)
At the start: 24 parts, among them J1 XT60PW-M_Horizontal, J10 SM02B-GHS-TB, J11 SM02B-GHS-TB, J12 SM02B-GHS-TB, J13 SM02B-GHS-TB, J14 SM02B-GHS-TB, J15 SM02B-GHS-TB, J16 SM02B-GHS-TB, J17 SM02B-GHS-TB, J18 RJ45, J19 Conn_01x02_Pin, J2 XT30PW-F_Horizontal, J20 RJ45, J22 Conn_01x04_Pin, J3 XT30PW-F_Horizontal, J4 XT30PW-F_Horizontal, J5 XT30PW-F_Horizontal, J6 XT30PW-F_Horizontal, J7 XT30PW-F_Horizontal, J8 XT30PW-F_Horizontal, J9 XT30PW-F_Horizontal, U1 BU33SD5WG-TR

Commit message: Ver1.1
Parts:
- added C16: 0.47μ, Capacitor_SMD:C_0603_1608Metric_Pad1.08x0.95mm_HandSolder, symbol Device:C
- added Q3: RD3L07BBGTL1, y-robo_footprint:TO252-3_ROM, symbol Transistor_FET:Q_NMOS_GDS
- added R5, R6: 100k, Resistor_SMD:R_0603_1608Metric_Pad0.98x0.95mm_HandSolder, symbol Device:R
Connections:
- net +24V: now also R5.1
- net GNDPWR: now also Q3.3 (S), R6.2; no longer J2.1 (-), J3.1 (-), J4.1 (-), J5.1 (-), J6.1 (-), J7.1 (-), J8.1 (-), J9.1 (-)
- new net: C16.2, Q3.1 (G), R5.2, R6.1
- new net GND1: C16.1, J2.1 (-), J3.1 (-), J4.1 (-), J5.1 (-), J6.1 (-), J7.1 (-), J8.1 (-), J9.1 (-), Q3.2 (D)
Other:
- moved on the sheet: J1, J10, J11, J12, J13, J14, J15, J16, J17, J2, J3, J4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
